Commit message: Add grasp and cell sequencer; correct belt nest; infer M1 Pro yaw; verified full cycle
Grasp: three gz DetachableJoint plugins (fork, cup, belt nest) emitted by
generate_cell_urdf.py, bridged as std_msgs/Empty on /wafer/<carrier>/attach
and /detach, plugin state back on /wafer/<carrier>/state. Two traps found
and documented in CLAUDE.md: gz-sim 8.11 attaches on start (attachRequested
defaults true), so go_home.py and the sequencer release all carriers first;
and parent links must survive URDF->SDF fixed-joint merging (m1pro_wrist_link,
pro600_link6, belt_carriage).

Sequencer: scripts/cell_sequencer.py runs yellow nest -> fork -> belt nest at
A -> belt A->B->C -> cup -> blue nest, every waypoint solved by IK from
cell_layout.py at start-up (seeded for one elbow branch), timing from the
2026-09-03 video as parameters (belt_speed, dwell_b, speed_scale, cycles),
step names on /cell/state as the Digital Shadow hook. --dry-run prints the
plan without a sim. scripts/record_frames.py saves timestamped frames.

Layout corrections:
- the belt carriage is the magenta C-nest (meshes/belt_nest.stl exported from
  meshes/Conveyor_Wafer_Holder.3MF, the print source, now in the repo); the
  flat bridge belt_holder.stl was a different part. Wafer rests on the rim,
  NEST_SEAT_Z = belt + 0.053
- M1 Pro base yaw -pi/2 by kinematic inference: with yaw 0 the fork cannot
  withdraw from the belt nest along -X as the video shows; with the carriage
  facing the bench front every cycle waypoint is reachable
- fork wafer seat at 147 mm from the wrist so the tine tips stop inside the
  nests' 57.5 mm free radius
- home poses re-solved on the belt-compatible elbow branch

Launch: verbose:=N argument; PRIME offload variables exported when the NVIDIA
module is loaded (GPU restored after the reboot, both gz processes on the
RTX 4060).

Verified 2026-09-04 00:43 on a clean simulator: all carriers report
attached/detached, wafer final pose (0.426, -0.166, 0.097) inside the blue
nest, 47 s sim time per cycle. Artefacts in docs/research_2026-09-03/
cycle_2026-09-04/. Cycle videos and the Gemini render copied into docs/.

Co-Authored-By: Claude Fable 5.1 <noreply@anthropic.com>

File: src/dobot_m1pro_description/urdf/dobot_m1pro.urdf.xacro (robot description, xacro)
@@ -241,9 +241,15 @@
     <origin xyz="0 0 0"/>
   </joint>
-  <!-- Wafer seat: on top of the blade, on the fork centreline. -->
+  <!-- Wafer seat: on top of the blade, on the fork centreline, 147 mm from
+       the wrist axis so the tine tips (177 mm) stop 30 mm past the wafer
+       centre. That keeps the tips inside the nests' free radius (57.5 mm, the
+       inner edge of the 2 mm ledges) so the blade can rise through the ledge
+       plane and lift the wafer; at 115 mm the tips sat 62 mm past centre,
+       under the ledge ring, and could not. ASSUMED - metrology
+       fork_support_geometry. -->
   <link name="${prefix}fork_seat"/>
   <joint name="${prefix}fork_seat_fixed" type="fixed">
     <parent link="${prefix}fork"/><child link="${prefix}fork_seat"/>
-    <origin xyz="0.1150 0 -0.0250"/>
+    <origin xyz="0.1470 0 -0.0250"/>
   </joint>
   <xacro:if value="$(arg use_gz_control)">

File: src/wafer_cell_bringup/urdf/cell.urdf (robot description, URDF)
Before this commit: robot wafer_cell, 21 links, 20 joints
Links:
- link belt_carriage: mass 0.15 -> 0.12; geometry collision mesh filename=package://wafer_cell_bringup/meshes/belt_nest.stl scale=0.001 0.001 0.001; visual mesh filename=package://wafer_cell_bringup/meshes/belt_nest.stl scale=0.001 0.001 0.001
Joints:
- joint m1pro_fork_seat_fixed: origin xyz=0.1150 0 -0.0250 -> xyz=0.1470 0 -0.0250
- joint m1pro_mount: origin xyz=-0.6 0.188 0.008 rpy=0.0 0.0 0.0 -> xyz=-0.6 0.188 0.008 rpy=0.0 0.0 -1.5707963267948966

File: src/wafer_cell_bringup/urdf/conveyor.urdf.xacro (robot description, xacro)
@@ -12,7 +12,14 @@
   Swapping in a real conveyor-system plugin later replaces THIS FILE ONLY;
   the sequencer talks to a joint either way.
-  Holder geometry is EXACT (customer STL): 180 mm along the belt x 70 mm
-  across x 45 mm tall, flat top with NO locating feature - the wafer is held
-  by friction alone, which is a real repeatability limit in the actual cell.
+  Carriage geometry (2026-09-04): the part that rides the belt is the magenta
+  C-NEST, print source ~/Downloads/Conveyor_Wafer_Holder.3MF, exported here as
+  meshes/belt_nest.stl (mm, Y up). Ring base r 29..45 mm, 3 mm thick; four
+  wall segments 53 mm tall with two 60-70 deg gaps on the mesh X axis (the
+  belt axis) for the fork tines and two small gaps on Z; a 3 mm ledge at
+  r 57.5..60.7 two mm below the rim, so the 127 mm wafer (r 63.5) actually
+  rests on the RIM TOP at 53 mm (NEST_SEAT_Z in cell_layout.py). Photographs
+  20260902_121240 and the cycle video show exactly this part on the belt with
+  its gap toward the M1 Pro. The earlier belt_holder.stl (180 x 70 x 45 flat
+  bridge) is a different part and is no longer used.
   ===========================================================================
 -->
@@ -22,5 +29,5 @@
   <xacro:arg name="controllers_file"
              default="$(find wafer_cell_bringup)/config/conveyor_controllers.yaml"/>
-  <xacro:property name="mesh" value="package://wafer_cell_bringup/meshes/belt_holder.stl"/>
+  <xacro:property name="mesh" value="package://wafer_cell_bringup/meshes/belt_nest.stl"/>
   <!-- travel: A = -0.25, C = +0.25. Limits are set WIDER (+/-0.30) so home
        never sits ON a limit - a joint initialised exactly at its limit latches
@@ -38,18 +45,22 @@
     </joint>
   </xacro:if>
+  <!-- mesh Y (up, -53..0) -> world Z via roll 90 deg; the bottom lands on
+       the belt surface with the +0.053 offset; mesh X (fork gaps) -> world X.
+       Collision is the mesh itself: the tines must pass between real wall
+       ends, a box would either block them or let them through walls. -->
   <link name="${prefix}carriage">
     <visual>
-      <origin xyz="0 0 0" rpy="1.5708 0 0"/>
+      <origin xyz="0 0 0.053" rpy="1.5708 0 0"/>
       <geometry><mesh filename="${mesh}" scale="0.001 0.001 0.001"/></geometry>
       <material name="holder_magenta"><color rgba="0.71 0.09 0.29 1"/></material>
     </visual>
     <collision>
-      <origin xyz="0 0 0.0405"/>
-      <geometry><box size="0.180 0.070 0.009"/></geometry>
+      <origin xyz="0 0 0.053" rpy="1.5708 0 0"/>
+      <geometry><mesh filename="${mesh}" scale="0.001 0.001 0.001"/></geometry>
     </collision>
     <inertial>
-      <origin xyz="0 0 0.030"/>
-      <mass value="0.15"/>
-      <inertia ixx="8.0e-5" ixy="0" ixz="0" iyy="4.5e-4" iyz="0" izz="4.9e-4"/>
+      <origin xyz="0 0 0.020"/>
+      <mass value="0.12"/>
+      <inertia ixx="1.2e-4" ixy="0" ixz="0" iyy="1.2e-4" iyz="0" izz="1.6e-4"/>
     </inertial>
   </link>

Commit message: Add Digital Shadow package with fake devices; primitive M1 Pro collisions; one cycle table
wafer_cell_shadow (new package):
- m1pro_bridge.py: Dobot port 30004, 1440-byte RealTimeData parsed at the
  offsets verified in Dobot-Arm/M1Pro-ROS commander.h (q_actual @432,
  robot_mode @24, DI @8); fake mode replays the ideal cycle in device units
- pro600_bridge.py: pymycobot ElephantRobot(host, port) get_angles/get_coords/
  get_digital_in; fake mode likewise
- plc_bridge.py: pycomm3 LogixDriver tag reads -> /shadow/plc/state (latched),
  belt_run, vacuum_on, belt_reverse; fake mode derives them from the cycle
- shadow_driver.py: streams /shadow/* joint states to the JTCs, dead-reckons
  the belt from belt_run x belt_speed with the reverse sign, applies grasp
  events after event_delay (the sim arm trails the real one by a horizon)
- launch/shadow.launch.py: source:=fake|real, record:=true (bag of /shadow/*),
  bridges:=false for replay; config/shadow.yaml with every UNKNOWN marked
- README with what is verified (packet layout, APIs) and what is not (IPs,
  port, tag names, joint signs/zeros, Z units)
- real-mode libraries in ~/venvs/wafer_shadow (system-site-packages venv)

Verified 2026-09-04: with fake devices the sim followed a full cycle and the
wafer ended in the blue nest (0.432, -0.156, 0.097); topics at 50/20 Hz.
Artefacts in docs/research_2026-09-03/shadow_2026-09-04/.

cell_plan.py: the cycle as one table (STEPS + build_waypoints + CycleState)
shared by cell_sequencer.py and the fake devices. Sequencer re-verified.

M1 Pro collisions: boxes/cylinder from the STL extents instead of 48k mesh
triangles. RTF headless 0.971 at rest / 0.984 in cycle (was 0.937 / 0.971);
earlier 0.5-0.75 figures were iGPU plus a stale server. rtf_2026-09-04.txt.

Co-Authored-By: Claude Fable 5.1 <noreply@anthropic.com>

File: src/dobot_m1pro_description/urdf/dobot_m1pro.urdf.xacro (robot description, xacro)
@@ -71,9 +71,15 @@
       </material>
     </visual>
-    <collision>
-      <origin xyz="0 0 0" rpy="0 0 0"/>
-      <geometry>
-        <mesh filename="${mesh_dir}/base_link.STL"/>
-      </geometry>
+    <!-- PRIMITIVE COLLISIONS (2026-09-04): the 25k-triangle base mesh and
+         the 5-10k arm meshes were the physics bottleneck (RTF 0.75 headless,
+         0.5 with GUI). Boxes sized from the STL extents; visuals unchanged.
+         base: casting z 0..0.06 (175 x 230), column z 0.06..0.688 (147 x 150) -->
+    <collision>
+      <origin xyz="0.0075 0 0.030" rpy="0 0 0"/>
+      <geometry><box size="0.175 0.230 0.060"/></geometry>
+    </collision>
+    <collision>
+      <origin xyz="-0.0015 0 0.374" rpy="0 0 0"/>
+      <geometry><box size="0.147 0.150 0.628"/></geometry>
     </collision>
   </link>
@@ -94,8 +100,6 @@
     </visual>
     <collision>
-      <origin xyz="0 0 0" rpy="0 0 0"/>
-      <geometry>
-        <mesh filename="${mesh_dir}/Link1.STL"/>
-      </geometry>
+      <origin xyz="0.108 0 0.1025" rpy="0 0 0"/>
+      <geometry><box size="0.130 0.100 0.205"/></geometry>
     </collision>
   </link>
@@ -115,9 +119,12 @@
       </material>
     </visual>
-    <collision>
-      <origin xyz="0 0 0" rpy="0 0 0"/>
-      <geometry>
-        <mesh filename="${mesh_dir}/Link2.STL"/>
-      </geometry>
+    <!-- root plate x -0.04..0.06 z 0..0.032; housing x 0.06..0.24 z 0..0.142 -->
+    <collision>
+      <origin xyz="0.010 0 0.016" rpy="0 0 0"/>
+      <geometry><box size="0.100 0.080 0.032"/></geometry>
+    </collision>
+    <collision>
+      <origin xyz="0.150 0 0.071" rpy="0 0 0"/>
+      <geometry><box size="0.180 0.080 0.142"/></geometry>
     </collision>
   </link>
@@ -137,9 +144,12 @@
       </material>
     </visual>
-    <collision>
-      <origin xyz="0 0 0" rpy="0 0 0"/>
-      <geometry>
-        <mesh filename="${mesh_dir}/Link3.STL"/>
-      </geometry>
+    <!-- elbow plate x -0.031..0.06 z -0.05..0.003; housing x 0.06..0.231 z -0.05..0.12 -->
+    <collision>
+      <origin xyz="0.0145 0 -0.0235" rpy="0 0 0"/>
+      <geometry><box size="0.091 0.062 0.053"/></geometry>
+    </collision>
+    <collision>
+      <origin xyz="0.1455 0 0.035" rpy="0 0 0"/>
+      <geometry><box size="0.171 0.064 0.170"/></geometry>
     </collision>
   </link>
@@ -163,8 +173,7 @@
          where it renders. -->
     <collision>
-      <origin xyz="0 0 0.08081" rpy="0 0 0"/>
-      <geometry>
-        <mesh filename="${mesh_dir}/Link4.STL"/>
-      </geometry>
+      <!-- the wrist shaft: mesh z -0.081..0.007 plus the 0.08081 offset -->
+      <origin xyz="0 0 0.044" rpy="0 0 0"/>
+      <geometry><cylinder radius="0.009" length="0.088"/></geometry>
     </collision>
   </link>

File: src/wafer_cell_bringup/urdf/cell.urdf (robot description, URDF)
Before this commit: robot wafer_cell, 21 links, 20 joints
Links:
- link m1pro_base_link: geometry collision box size=0.147 0.150 0.628; collision box size=0.175 0.230 0.060
- link m1pro_forearm_link: geometry collision box size=0.091 0.062 0.053; collision box size=0.171 0.064 0.170
- link m1pro_upper_arm_link: geometry collision box size=0.100 0.080 0.032; collision box size=0.180 0.080 0.142
- link m1pro_wrist_link: geometry collision cylinder length=0.088 radius=0.009; visual mesh filename=package://dobot_m1pro_description/meshes/Link4.STL
- link m1pro_z_carriage_link: geometry collision box size=0.130 0.100 0.205; visual mesh filename=package://dobot_m1pro_description/meshes/Link1.STL

Commit message: Fix wafer seating end to end; belt holder STL, Pro 600 colour, blue nest, close-up cameras
Owner's five corrections (2026-09-04 evening):
- Belt carriage is meshes/belt_holder.stl ridden plate-down with its posts up;
  the Ø124 C-nest 3MF and belt_nest.stl were the wrong part and are removed.
- Pro 600 recoloured from bright white to a warm light grey, link6 darker.
- Blue tower turned to open -X like the yellow one (owner's instruction; the
  2026-09-02 photo showed +X, noted in cell_layout.py).
- Wafer Ø127 checked against all three nests: tower step wall r 64, holder
  lip r 64, both 0.5 mm radial clearance; wafer collision r 63.0 under a
  63.5 visual to stand in for print chamfers.
- Wafer now seats: five root causes found with streamed pose logs and fixed.
  * Fork approach point clipped the wafer rim (tip overhang 30 mm + radius
    63.5 > 90 mm): now retreat at carry height, 115 mm back, descend, slide in
    4 mm under, lift 1 mm so the wafer rests on the tines, then weld.
  * Third M1 Pro vendor defect: elbow frame rolled -1 deg with the axis
    tilted; the fork came out rolled 1.000 deg. Fixed in the xacro.
  * Pro 600 cup collision ran 9 mm past the tip frame the plan steers to and
    rammed the wafer through the holder before the joint formed.
  * Joint-space cup descents bowed 5 mm sideways over 120 mm; 20 mm near_*
    waypoints make the last stretch straight.
  * A free 5.5 mm drop into the holder kicked the disc in 3 of 5 runs (welded
    standing 23 deg for the ride). NEST_SEAT places it on the seat with
    set_pose (wafer_seat.py): a declared stand-in until the owner says how the
    real fork lowers the wafer past the 45 mm posts.
- Controllers: goal bands 0.0005 rad / 0.3 mm, goal_time 3 s.
- Four close-up cameras (/detail_yellow_cam, /detail_belt_cam,
  /detail_beltc_cam, /detail_blue_cam) for millimetre seating checks.
- Shadow package follows the same cycle table (NEST_SEAT, near_* steps).

Verified: full cycle completes; the wafer rides the belt seated to 0.2 mm and
ends in the blue nest 0.3 / 0.5 mm off centre at ledge height; check_extents
clean. Traps recorded in CLAUDE.md; HANDOVER, PROJECT_CONTEXT and the
research review updated. Bullet collision detector tried and rejected
(convex-hulls the C-nests).

Co-Authored-By: Claude Fable 5.1 <noreply@anthropic.com>

File: src/dobot_m1pro_description/urdf/dobot_m1pro.urdf.xacro (robot description, xacro)
@@ -194,9 +194,17 @@
     <dynamics damping="1.0" friction="0.5"/>
   </joint>
+  <!-- VENDOR DEFECT FIXED (3): upstream rolls the forearm frame by -1 deg
+       (rpy -0.017453) and tilts the axis back by +1 deg (0 0.017452 -0.99985),
+       so the elbow axis is vertical but every downstream frame - the wrist
+       axis and the fork blade - is rolled 1.000 deg (measured by FK). A SCARA
+       wrist is vertical; that roll tilted the carried wafer 2.2 mm edge to
+       edge. Roll removed, axis exactly vertical; the 1.96 deg yaw offset of
+       the elbow zero is kept (it belongs to the joint-angle mapping, see the
+       shadow's offset parameters). -->
   <joint name="${prefix}elbow" type="revolute">
-    <origin xyz="0.2 0 0" rpy="-0.017453 0 0.034228"/>
+    <origin xyz="0.2 0 0" rpy="0 0 0.034228"/>
     <parent link="${prefix}upper_arm_link"/>
     <child link="${prefix}forearm_link"/>
-    <axis xyz="0 0.017452 -0.99985"/>
+    <axis xyz="0 0 -1"/>
     <limit lower="-2.356194" upper="2.356194" effort="204.0" velocity="3.14"/>
     <dynamics damping="1.0" friction="0.5"/>

File: src/mycobot_pro600_description/urdf/mycobot_pro600.urdf.xacro (robot description, xacro)
@@ -69,4 +69,5 @@
       <origin xyz="0 0 0" rpy="0 0 0"/>
       <geometry><mesh filename="${mesh_dir}/base.stl"/></geometry>
+      <material name="pro600_body"><color rgba="0.82 0.82 0.80 1"/></material>
     </visual>
     <collision>
@@ -82,4 +83,5 @@
       <origin xyz="0 0 0" rpy="0 0 3.1415926"/>
       <geometry><mesh filename="${mesh_dir}/link1.stl"/></geometry>
+      <material name="pro600_body"><color rgba="0.82 0.82 0.80 1"/></material>
     </visual>
     <collision>
@@ -96,4 +98,5 @@
       <origin xyz="0 0 -0.080" rpy="3.1415926 0 3.1415926"/>
       <geometry><mesh filename="${mesh_dir}/link2.stl"/></geometry>
+      <material name="pro600_body"><color rgba="0.82 0.82 0.80 1"/></material>
     </visual>
     <collision>
@@ -109,4 +112,5 @@
       <origin xyz="0 0 -0.0855" rpy="3.1415926 0 3.1415926"/>
       <geometry><mesh filename="${mesh_dir}/link3.stl"/></geometry>
+      <material name="pro600_body"><color rgba="0.82 0.82 0.80 1"/></material>
     </visual>
     <collision>
@@ -122,4 +126,5 @@
       <origin xyz="0 0 0" rpy="0 3.1415926 0"/>
       <geometry><mesh filename="${mesh_dir}/link4.stl"/></geometry>
+      <material name="pro600_body"><color rgba="0.82 0.82 0.80 1"/></material>
     </visual>
     <collision>
@@ -135,4 +140,5 @@
       <origin xyz="0 0 0" rpy="0 0 1.5707"/>
       <geometry><mesh filename="${mesh_dir}/link5.stl"/></geometry>
+      <material name="pro600_body"><color rgba="0.82 0.82 0.80 1"/></material>
     </visual>
     <collision>
@@ -148,5 +154,5 @@
       <origin xyz="0.03 0 0" rpy="0 -1.5707 0"/>
       <geometry><mesh filename="${mesh_dir}/link6.stl"/></geometry>
-      <material name="pro600_grey"><color rgba="0.5 0.5 0.5 1"/></material>
+      <material name="pro600_grey"><color rgba="0.55 0.56 0.58 1"/></material>
     </visual>
     <collision>
@@ -223,7 +229,11 @@
       <material name="cup_blue"><color rgba="0.11 0.40 0.78 1"/></material>
     </visual>
-    <collision>
-      <origin xyz="0 0 0.0300" rpy="0 0 0"/>
-      <geometry><cylinder radius="0.0180" length="0.0600"/></geometry>
+    <!-- Collision ENDS AT THE TIP FRAME (z 0.051). It used to run to z 0.060,
+         9 mm past the tip the plan steers to, and rammed the wafer 17 mm
+         down through the belt holder before the joint was made (cycle 11,
+         2026-09-04). -->
+    <collision>
+      <origin xyz="0 0 0.0255" rpy="0 0 0"/>
+      <geometry><cylinder radius="0.0180" length="0.0510"/></geometry>
     </collision>
     <inertial>

File: src/wafer_cell_bringup/urdf/cell.urdf (robot description, URDF)
Before this commit: robot wafer_cell, 21 links, 20 joints
Links:
- link belt_carriage: geometry collision mesh filename=package://wafer_cell_bringup/meshes/belt_holder.stl scale=0.001 0.001 0.001; visual mesh filename=package://wafer_cell_bringup/meshes/belt_holder.stl scale=0.001 0.001 0.001
- link pro600_cup: geometry collision cylinder length=0.0510 radius=0.0180; visual cylinder length=0.0160 radius=0.0180
Joints:
- joint m1pro_elbow: axis 0 0.017452 -0.99985 -> 0 0 -1; origin xyz=0.2 0 0 rpy=-0.017453 0 0.034228 -> xyz=0.2 0 0 rpy=0 0 0.034228

File: src/wafer_cell_bringup/urdf/conveyor.urdf.xacro (robot description, xacro)
@@ -12,14 +12,15 @@
   Swapping in a real conveyor-system plugin later replaces THIS FILE ONLY;
   the sequencer talks to a joint either way.
-  Carriage geometry (2026-09-04): the part that rides the belt is the magenta
-  C-NEST, print source ~/Downloads/Conveyor_Wafer_Holder.3MF, exported here as
-  meshes/belt_nest.stl (mm, Y up). Ring base r 29..45 mm, 3 mm thick; four
-  wall segments 53 mm tall with two 60-70 deg gaps on the mesh X axis (the
-  belt axis) for the fork tines and two small gaps on Z; a 3 mm ledge at
-  r 57.5..60.7 two mm below the rim, so the 127 mm wafer (r 63.5) actually
-  rests on the RIM TOP at 53 mm (NEST_SEAT_Z in cell_layout.py). Photographs
-  20260902_121240 and the cycle video show exactly this part on the belt with
-  its gap toward the M1 Pro. The earlier belt_holder.stl (180 x 70 x 45 flat
-  bridge) is a different part and is no longer used.
+  Carriage geometry (corrected by the owner 2026-09-04): the part that rides
+  the belt is meshes/belt_holder.stl, a 180 x 70 mm PLATE (3 mm) that lies
+  on the belt with two 45 mm POSTS rising at the belt-axis ends. Each post's
+  inner face is a concave arc of radius 57.5 mm (the "curve cuts"); a ring
+  seat at 43 mm and a 2 mm lip of radius ~64 mm hold the 127 mm wafer
+  (photo reference_photos_4/20260902_121240). The STL is modelled plate-up
+  (plate at file y 42..45, posts hanging to y 0), so it is rolled -90 deg
+  about X and lifted 45 mm: plate on the belt, posts up.
+  A fork blade under the wafer cannot pass a post along the belt, so the
+  fork releases the wafer from just above the posts and it drops ~7 mm
+  into the lip (cell_plan.py). NEST_SEAT_Z / HOLDER_POST_TOP in cell_layout.py.
   ===========================================================================
 -->
@@ -29,5 +30,5 @@
   <xacro:arg name="controllers_file"
              default="$(find wafer_cell_bringup)/config/conveyor_controllers.yaml"/>
-  <xacro:property name="mesh" value="package://wafer_cell_bringup/meshes/belt_nest.stl"/>
+  <xacro:property name="mesh" value="package://wafer_cell_bringup/meshes/belt_holder.stl"/>
   <!-- travel: A = -0.25, C = +0.25. Limits are set WIDER (+/-0.30) so home
        never sits ON a limit - a joint initialised exactly at its limit latches
@@ -45,16 +46,16 @@
     </joint>
   </xacro:if>
-  <!-- mesh Y (up, -53..0) -> world Z via roll 90 deg; the bottom lands on
-       the belt surface with the +0.053 offset; mesh X (fork gaps) -> world X.
-       Collision is the mesh itself: the tines must pass between real wall
-       ends, a box would either block them or let them through walls. -->
+  <!-- file frame: Y is the height axis with the plate at the TOP (y 42..45).
+       roll -90 deg maps file +Y to world -Z (plate down, posts up), file Z
+       (70 mm) to world Y across the belt; +0.045 puts the plate on the belt.
+       Collision is the mesh: the wafer must land inside real posts and lip. -->
   <link name="${prefix}carriage">
     <visual>
-      <origin xyz="0 0 0.053" rpy="1.5708 0 0"/>
+      <origin xyz="0 0 0.045" rpy="-1.5708 0 0"/>
       <geometry><mesh filename="${mesh}" scale="0.001 0.001 0.001"/></geometry>
       <material name="holder_magenta"><color rgba="0.71 0.09 0.29 1"/></material>
     </visual>
     <collision>
-      <origin xyz="0 0 0.053" rpy="1.5708 0 0"/>
+      <origin xyz="0 0 0.045" rpy="-1.5708 0 0"/>
       <geometry><mesh filename="${mesh}" scale="0.001 0.001 0.001"/></geometry>
     </collision>
