Commit message: Apply interim photo-derived layout; single source of poses in cell_layout.py
Owner's instruction 2026-09-03: apply the layout estimated from the
rectified overhead photograph (docs/research_2026-09-03, +/-20 mm) as an
interim until measurements land.

Layout changes (world frame, metres):
- yellow nest (-0.353, -0.162) opening toward -X; blue nest (0.430, -0.153)
  opening toward +X (directions verified from photos; both were +Y)
- conveyor mesh yawed 180 deg so the stepper motor sits at the -X rear
  corner as photographed; bbox centred on the real centreline y = +0.135
- M1 Pro base (-0.600, +0.188), Pro 600 base (+0.600, +0.200), plates
  resized to the photographed outlines; both base YAWS unchanged, unmeasured
- belt waypoints A -0.14, B +0.03, C +0.20 (holder at rest / video)
- wafer spawns on the yellow nest's top shelf at the new position

Structure:
- new scripts/cell_layout.py holds every pose, limit and the home pose;
  generate_cell_urdf.py, go_home.py, check_extents.py and cell.launch.py
  import it. wafer_cell.sdf mirrors the numbers and check_extents.py now
  exits non-zero if the two disagree
- new scripts/solve_home_poses.py: numerical IK on cell.urdf for rest and
  pick poses with limit margins; rest poses re-solved for this layout
  (fork hovering above the yellow nest pointing +X, cup above point C)
- cell.urdf regenerated

Verified headless on the Intel iGPU after killing two stale gz servers:
4/4 controllers active, 11/11 joints on the solved home, 0 parts off the
bench, both camera captures (docs/cell_layout.png, docs/cell_plan.png).
Reach check: fork reaches under the wafer at the yellow nest and over the
holder at A; cup reaches C and the blue nest.

Docs: CLAUDE.md, PROJECT_CONTEXT.md section 14, HANDOVER.md and README.md
updated for the interim layout, the found reference assets, and the
headless-orphan detection pattern.

Co-Authored-By: Claude Fable 5.1 <noreply@anthropic.com>

File: src/wafer_cell_bringup/urdf/cell.urdf (robot description, URDF)
Before this commit: robot wafer_cell, 21 links, 20 joints
Joints:
- joint belt_mount: origin xyz=0.0 0.13 0.06265 rpy=0 0 0 -> xyz=0.0 0.135 0.06265 rpy=0.0 0.0 0.0
- joint m1pro_mount: origin xyz=-0.56 0.15 0.008 rpy=0 0 0.0 -> xyz=-0.6 0.188 0.008 rpy=0.0 0.0 0.0
- joint pro600_mount: origin xyz=0.62 0.18 0.008 rpy=0 0 3.14159 -> xyz=0.6 0.2 0.008 rpy=0.0 0.0 3.141592653589793

Commit message: Fork turns 90 deg and enters the belt holder across the belt; holder back along the belt
Owner's correction (with a picture): the holder sits with its 180 mm side
ALONG the belt, posts at the belt-axis ends, as first built. What the
videos show is the FORK's motion: during the transfer from the yellow nest
the wrist turns the fork 90 deg so it enters the holder ACROSS the belt from
the bench front, between the two posts, sets the wafer on the seats and
backs out underneath. My previous commit had turned the holder instead.

- conveyor.urdf.xacro: holder yaw reverted (roll -90 only); header states
  the orientation and the fork's entry; belt joint lower limit -0.32.
- cell_layout.py: BELT_A -0.25 (holder loads beside the column with its end
  at the belt's end, as in the video; the photo's -0.14 is out of the
  M1 Pro's reach for an across-belt entry, checked by IK scan).
- cell_plan.py: FORK_AX_BELT (blade pointing +Y) for the belt waypoints,
  APPROACH_BELT 0.08 from the front; set-down / release / drop-blade /
  retreat sequence kept.
- detail_belt_cam re-aimed from behind the belt so the blade is seen
  arriving between the posts.
- Docs corrected again: CLAUDE.md, HANDOVER, PROJECT_CONTEXT, research
  review, verification captures (cycle 16, hand-off from the rear).

Verified: full cycle completes; set-down at seat height, 0.0 mm / 0.0 deg;
rides seated; ends at the blue nest centre; check_extents clean.

Co-Authored-By: Claude Fable 5.1 <noreply@anthropic.com>

File: src/wafer_cell_bringup/urdf/cell.urdf (robot description, URDF)
Before this commit: robot wafer_cell, 21 links, 20 joints
Joints:
- joint belt_travel: limit lower=-0.3 upper=0.3 effort=200.0 velocity=0.5 -> lower=-0.32 upper=0.3 effort=200.0 velocity=0.5

File: src/wafer_cell_bringup/urdf/conveyor.urdf.xacro (robot description, xacro)
@@ -19,10 +19,12 @@
   (plate at file y 42..45, posts hanging to y 0), so it is rolled -90 deg
   about X and lifted 45 mm: plate on the belt, posts up.
-  ORIENTATION (owner's hand-off video, 2026-09-04 evening): the plate's
-  180 mm side lies ACROSS the belt and the posts stand at the belt's FRONT
-  and REAR, overhanging the rails ~25 mm each side. The fork slides the
-  wafer in ALONG the belt between the posts, sets it on the seats and backs
-  out underneath (cell_plan.py). An earlier build had the posts at the
-  belt-axis ends, which made that hand-off impossible and forced a drop.
+  ORIENTATION (owner, 2026-09-04 late evening, with a picture): the plate's
+  180 mm side lies ALONG the belt, the posts stand at the belt-axis ends.
+  The fork does NOT enter along the belt: during the transfer from the
+  yellow nest the wrist turns the fork 90 deg so it enters ACROSS the belt
+  from the front, between the two posts, sets the wafer on the seats and
+  backs out underneath (owner's videos; cell_plan.py). I twice got this
+  wrong (posts across the belt, then a drop stand-in): read the videos
+  for the FORK's motion, not only the fixture's.
   NEST_SEAT_Z / HOLDER_POST_TOP in cell_layout.py.
   ===========================================================================
@@ -37,5 +39,5 @@
        never sits ON a limit - a joint initialised exactly at its limit latches
        and then silently ignores every command. -->
-  <xacro:property name="lo"   value="-0.30"/>
+  <xacro:property name="lo"   value="-0.32"/>   <!-- load position -0.25 keeps the 0.05 init margin -->
   <xacro:property name="hi"   value="0.30"/>
   <xacro:property name="home" value="-0.25"/>
@@ -50,17 +52,16 @@
   </xacro:if>
   <!-- file frame: Y is the height axis with the plate at the TOP (y 42..45).
-       roll -90 deg maps file +Y to world -Z (plate down, posts up); the yaw
-       of +90 deg then puts the file X (180 mm, posts at its ends) ACROSS the
-       belt (world Y) and the file Z (70 mm) along it; +0.045 puts the plate
-       on the belt. Collision is the mesh: the wafer must land inside real
-       posts and lip. -->
+       roll -90 deg maps file +Y to world -Z (plate down, posts up), file X
+       (180 mm, posts at its ends) stays along the belt (world X) and file Z
+       (70 mm) goes across it; +0.045 puts the plate on the belt.
+       Collision is the mesh: the wafer must land inside real posts and lip. -->
   <link name="${prefix}carriage">
     <visual>
-      <origin xyz="0 0 0.045" rpy="-1.5708 0 1.5708"/>
+      <origin xyz="0 0 0.045" rpy="-1.5708 0 0"/>
       <geometry><mesh filename="${mesh}" scale="0.001 0.001 0.001"/></geometry>
       <material name="holder_magenta"><color rgba="0.71 0.09 0.29 1"/></material>
     </visual>
     <collision>
-      <origin xyz="0 0 0.045" rpy="-1.5708 0 1.5708"/>
+      <origin xyz="0 0 0.045" rpy="-1.5708 0 0"/>
       <geometry><mesh filename="${mesh}" scale="0.001 0.001 0.001"/></geometry>
     </collision>

Commit message: Centre the belt carriage on the belt's running surface; cycle_recording_09_04_2026.mp4
Owner's GUI screenshot showed the holder riding 30 mm off the belt's centre.
The conveyor mesh's bounding box includes the motor housing on the rear
side, so its centre (y 0.135) is not the belt. A cross-section of
dobot_conveyor.stl at mid-length puts the belt band at world y 0.045..0.165.

- cell_layout.py: BELT_SURFACE_Y 0.105 and CARRIAGE_XYZ; the conveyor xacro
  is placed at CARRIAGE_XYZ, BELT_XYZ only anchors the mesh.
- cell_plan.py and solve_home_poses.py: belt targets on BELT_SURFACE_Y.
- Both belt cameras shifted with the carriage.
- CLAUDE.md trap and HANDOVER note; verification recording replaced.

Verified: extents clean, every belt waypoint reachable (<= 0.8 mm), full
cycle recorded end to end, holder centred on the belt in the plan view.

Co-Authored-By: Claude Fable 5.1 <noreply@anthropic.com>

File: src/wafer_cell_bringup/urdf/cell.urdf (robot description, URDF)
Before this commit: robot wafer_cell, 21 links, 20 joints
Joints:
- joint belt_mount: origin xyz=0.0 0.135 0.06265 rpy=0.0 0.0 0.0 -> xyz=0.0 0.105 0.06265 rpy=0.0 0.0 0.0

Commit message: Band-split the belt holder collision mesh as well
belt_holder_collision.stl (8 mm bands) replaces the raw STL as the carriage
collision; visual unchanged; cell.urdf regenerated. Headless 1 ms: overall
RTF 0.98, ride seated at 43.7 mm, end pose (0.4300, -0.1530, 0.0997)
identical to the approved result; check_extents clean.

Co-Authored-By: Claude Fable 5.1 <noreply@anthropic.com>

File: src/wafer_cell_bringup/urdf/cell.urdf (robot description, URDF)
Before this commit: robot wafer_cell, 21 links, 20 joints
Links:
- link belt_carriage: geometry collision mesh filename=package://wafer_cell_bringup/meshes/belt_holder_collision.s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 scale=0.001 0.001 0.001; visual mesh filename=package://wafer_cell_bringup/meshes/belt_holder.stl scale=0.001 0.001 0.001

File: src/wafer_cell_bringup/urdf/conveyor.urdf.xacro (robot description, xacro)
@@ -37,4 +37,7 @@
              default="$(find wafer_cell_bringup)/config/conveyor_controllers.yaml"/>
   <xacro:property name="mesh" value="package://wafer_cell_bringup/meshes/belt_holder.stl"/>
+  <!-- collision: the same surface cut into 8 mm bands (scripts/split_collision_mesh.py)
+       so the ODE mesh tree culls by height; see the tower note in the world file -->
+  <xacro:property name="mesh_collision" value="package://wafer_cell_bringup/meshes/belt_holder_collision.stl"/>
   <!-- travel: A = -0.25, C = +0.25. Limits are set WIDER (+/-0.30) so home
        never sits ON a limit - a joint initialised exactly at its limit latches
@@ -65,5 +68,5 @@
     <collision>
       <origin xyz="0 0 0.045" rpy="-1.5708 0 0"/>
-      <geometry><mesh filename="${mesh}" scale="0.001 0.001 0.001"/></geometry>
+      <geometry><mesh filename="${mesh_collision}" scale="0.001 0.001 0.001"/></geometry>
     </collision>
     <inertial>

Commit message: Taught-path cycle and layout from the PLC programmer's taught poses
Adopt Alonso's taught M1 Pro and Pro 600 poses and fix the two divergences
from the bench:

- cell_plan: the M1 rest pose sits 86.6 mm straight above the approach
  point, 139 mm insert, 41.4 mm lift, wrist turn of 94.16 deg (his R values),
  arrival directly above the carrier, vertical set-down, J1-only swing-out
  (-19.75 deg, sign found by FK), 75.5 mm lift-out; Pro 600 descends 28 mm
  at the pick and 37 mm at the place with the traverse between those heights.
- The belt no longer returns inside the cycle: MANUAL_RETURN_A follows
  CYCLE_DONE as a declared stand-in for the hand carry.
- cell_layout: the M1 side placed from his Cartesian values (wrist axis in
  the J1 frame; 200+200 mm links confirmed by his J1 readings), the Pro 600
  side from his three distances with the blue nest on the yellow's line, the
  carrier kept at its 09-04 place on the belt by shifting the conveyor 20 mm.
  The photo layout had the conveyor and pick tower 55-70 mm too far forward.
- Stations are belt joint positions; BELT_A_X / BELT_C_X are world x.
- World file: conveyor mesh and Pro 600 plate follow the layout, the M1's
  duplicate plate removed, cameras re-aimed; check_extents now mirrors the
  conveyor mesh and the plate so a belt move cannot leave them behind again.
- Shadow package: step renames, MANUAL_RETURN_A, and the task shadow's
  first-idle gating counts played segments (it skipped the IDLE segment
  when the fake PLC's Pro 600 job outlasted the simulated one).
- tools/cycle_check: streamed pose check of one headless cycle.

Verified headless with the streamed pose log (seated 43.8 mm, 0.0 mm offset,
tilt < 0.3 deg through swing-out, lift-out and both belt moves; place at
(0.407, -0.230, 0.0997)), Level 1 against fake_plc end to end, six-camera
captures, and one cycle in the GUI reviewed by the owner.

Co-Authored-By: Claude Fable 5.1 <noreply@anthropic.com>

File: src/wafer_cell_bringup/urdf/cell.urdf (robot description, URDF)
Before this commit: robot wafer_cell, 21 links, 20 joints
Joints:
- joint belt_mount: origin xyz=0.0 0.105 0.06265 rpy=0.0 0.0 0.0 -> xyz=0.02 0.161 0.06265 rpy=0.0 0.0 0.0
- joint m1pro_mount: origin xyz=-0.6 0.188 0.008 rpy=0.0 0.0 -1.5707963267948966 -> xyz=-0.609 0.204 0.0 rpy=0.0 0.0 -1.5707963267948966
- joint pro600_mount: origin xyz=0.6 0.2 0.008 rpy=0.0 0.0 3.141592653589793 -> xyz=0.6 0.124 0.008 rpy=0.0 0.0 3.141592653589793

Commit message: Telemetry mode with both joint mappings; Pro 600 base yaw fitted from the recordings
Real-to-sim as the TA defined it on 2026-09-11: the two arms follow their own
joint telemetry, everything else is a prop.

- cell.launch.py telemetry:=true spawns JointGroupPositionControllers for both
  arms instead of the trajectory controllers; go_home only releases the wafer
  welds (--release-only); the arms hold their URDF initial values, which are
  the real HOME through the mappings.
- tools/replay_telemetry.py replays the owner's first bench recordings (M1 Pro
  port 30004 log, Pro 600 UDP 5005 log) as forward-position commands and as the
  sensor_msgs/JointState contract on /telemetry/<robot>/joint_states, parks the
  wafer, and reports the tracking error.
- M1 Pro mapping verified on the full recording against every taught waypoint
  (0.1 deg): shoulder = J1, elbow = -J2 + 1.961 deg, wrist = J4 - 17.54 deg,
  z_lift = J3 + 24.4 mm. The sim already used the real elbow configuration.
- Pro 600 mapping fitted on his four confirmed pose pairs with the cup direction
  in the score: joint2 and joint4 = his + 90 deg, the rest unchanged; his
  controller frame is the vendor URDF base frame; his Cartesian table is the
  cup tip, 31 mm above the model's cup (real cup assembly ~3 cm longer).
- PRO600_YAW -92.5 deg (was an unmeasured pi): his mapped poses land on C,
  the blue nest and his HOME within 4 mm. The Pro 600 rest pose is now his HOME
  angles through the mapping.
- Measurement sheet regenerated for the moved Pro 600 footprint.

Verified: dry run, extents, the sim's own cycle (place at the blue nest, seating
43.8 mm, tilt < 0.2 deg), and both recordings replayed in telemetry mode from
HOME back to HOME with ~3 deg worst latency error.

Co-Authored-By: Claude Fable 5.1 <noreply@anthropic.com>

File: src/wafer_cell_bringup/urdf/cell.urdf (robot description, URDF)
Before this commit: robot wafer_cell, 21 links, 20 joints
Joints:
- joint pro600_mount: origin xyz=0.6 0.124 0.008 rpy=0.0 0.0 3.141592653589793 -> xyz=0.6 0.124 0.008 rpy=0.0 0.0 -1.6144
